File: ringRemote.sch (EAGLE design)
At the start: 25 parts, among them J1 AMPHENOL_10118192-0001LFAMPHE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, Y1 32.768kHz

Commit message: made rough layout of board; swapped some pins for pushbuttons in sch (to atbtlc); understood programming workflow a bit better (likely using SWD instead of i2c)
Connections:
- net N$8 renamed PB3
- net N$9 renamed PB4
- removed net N$6: R4.1, U$1.SWDIOALT
- removed net N$7: R1.1, U$1.SWDCLKALT
- new net I2C0_SCL: U$1.SWDIOALT
- new net I2C0_SDA: U$1.SWDCLKALT
- new net PB1: R1.1, U$2.LP_GPIO_14
- new net PB2: R4.1, U$2.LP_GPIO_15
- new net SWDCLK: U$1.SWDCLK
- new net SWDIO: U$1.SWDIO
Other:
- note added: "rename swdclkalt, etc. back to p0..."
- moved on the sheet: R1, R4, R5, R6
Changed lines of the file:
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@@
 can I be lazy and not include
 c5 and c6?</text>
-<text x="38.1" y="15.24" size="1.27" layer="97" align="bottom-right">not adding a sch part,
+<text x="48.26" y="101.6" size="1.27" layer="97" align="bottom-right">not adding a sch part,
 but there are hypothetical
 switches here. will probably
@@
 filament under (as carrier) then pot
 with conductive glue</text>
+<text x="5.08" y="55.88" size="1.27" layer="97">rename swdclkalt, etc. back to p0...</text>
 </plain>
 <instances>
@@
 <instance part="R3" gate="G$1" x="99.06" y="30.48" rot="R270"/>
 <instance part="GND9" gate="G$1" x="99.06" y="12.7"/>
-<instance part="R1" gate="G$1" x="30.48" y="55.88" rot="R180"/>
-<instance part="R4" gate="G$1" x="43.18" y="53.34" rot="R180"/>
-<instance part="R5" gate="G$1" x="30.48" y="38.1" rot="R180"/>
-<instance part="R6" gate="G$1" x="43.18" y="35.56" rot="R180"/>
-<instance part="GND3" gate="G$1" x="38.1" y="30.48"/>
-<instance part="GND10" gate="G$1" x="25.4" y="33.02"/>
-<instance part="GND11" gate="G$1" x="25.4" y="50.8"/>
-<instance part="GND12" gate="G$1" x="38.1" y="48.26"/>
-<instance part="SUPPLY4" gate="G$1" x="25.4" y="60.96"/>
-<instance part="SUPPLY5" gate="G$1" x="38.1" y="58.42"/>
-<instance part="SUPPLY6" gate="G$1" x="25.4" y="43.18"/>
-<instance part="SUPPLY7" gate="G$1" x="38.1" y="40.64"/>
+<instance part="R1" gate="G$1" x="33.02" y="152.4" rot="R180"/>
+<instance part="R4" gate="G$1" x="45.72" y="149.86" rot="R180"/>
+<instance part="R5" gate="G$1" x="33.02" y="129.54" rot="R180"/>
+<instance part="R6" gate="G$1" x="45.72" y="127" rot="R180"/>
+<instance part="GND3" gate="G$1" x="40.64" y="121.92"/>
+<instance part="GND10" gate="G$1" x="27.94" y="124.46"/>
+<instance part="GND11" gate="G$1" x="27.94" y="147.32"/>
+<instance part="GND12" gate="G$1" x="40.64" y="144.78"/>
+<instance part="SUPPLY4" gate="G$1" x="27.94" y="157.48"/>
+<instance part="SUPPLY5" gate="G$1" x="40.64" y="154.94"/>
+<instance part="SUPPLY6" gate="G$1" x="27.94" y="134.62"/>
+<instance part="SUPPLY7" gate="G$1" x="40.64" y="132.08"/>
 <instance part="FRAME1" gate="G$1" x="0" y="0"/>
 <instance part="FRAME1" gate="V" x="147.32" y="0"/>
@@
 <pinref part="R6" gate="G$1" pin="2"/>
 <pinref part="GND3" gate="G$1" pin="3.3V"/>
-<wire x1="38.1" y1="35.56" x2="38.1" y2="33.02" width="0.1524" layer="91"/>
+<wire x1="40.64" y1="127" x2="40.64" y2="124.46" width="0.1524" layer="91"/>
 </segment>
 <segment>
 <pinref part="R5" gate="G$1" pin="2"/>
 <pinref part="GND10" gate="G$1" pin="3.3V"/>
-<wire x1="25.4" y1="38.1" x2="25.4" y2="35.56" width="0.1524" layer="91"/>
+<wire x1="27.94" y1="129.54" x2="27.94" y2="127" width="0.1524" layer="91"/>
 </segment>
 <segment>
 <pinref part="R1" gate="G$1" pin="2"/>
 <pinref part="GND11" gate="G$1" pin="3.3V"/>
-<wire x1="25.4" y1="55.88" x2="25.4" y2="53.34" width="0.1524" layer="91"/>
+<wire x1="27.94" y1="152.4" x2="27.94" y2="149.86" width="0.1524" layer="91"/>
 </segment>
 <segment>
 <pinref part="R4" gate="G$1" pin="2"/>
 <pinref part="GND12" gate="G$1" pin="3.3V"/>
-<wire x1="38.1" y1="53.34" x2="38.1" y2="50.8" width="0.1524" layer="91"/>
+<wire x1="40.64" y1="149.86" x2="40.64" y2="147.32" width="0.1524" layer="91"/>
 </segment>
 </net>
@@
 </segment>
 </net>
-<net name="N$6" class="0">
-<segment>
-<pinref part="R4" gate="G$1" pin="1"/>
-<pinref part="U$1" gate="G$1" pin="SWDIOALT"/>
-<wire x1="48.26" y1="53.34" x2="50.8" y2="53.34" width="0.1524" layer="91"/>
-</segment>
-</net>
-<net name="N$7" class="0">
-<segment>
-<pinref part="U$1" gate="G$1" pin="SWDCLKALT"/>
-<wire x1="50.8" y1="55.88" x2="35.56" y2="55.88" width="0.1524" layer="91"/>
-<pinref part="R1" gate="G$1" pin="1"/>
-</segment>
-</net>
-<net name="N$8" class="0">
-<segment>
-<pinref part="U$1" gate="G$1" pin="P0.3"/>
-<pinref part="R5" gate="G$1" pin="1"/>
-<wire x1="50.8" y1="38.1" x2="35.56" y2="38.1" width="0.1524" layer="91"/>
-</segment>
-</net>
-<net name="N$9" class="0">
-<segment>
-<pinref part="U$1" gate="G$1" pin="P0.2"/>
-<pinref part="R6" gate="G$1" pin="1"/>
-<wire x1="50.8" y1="35.56" x2="48.26" y2="35.56" width="0.1524" layer="91"/>
-</segment>
-</net>
 <net name="MAXRST" class="0">
 <segment>
@@
 </segment>
 </net>
+<net name="PB1" class="0">
+<segment>
+<pinref part="U$2" gate="G$1" pin="LP_GPIO_14"/>
+<wire x1="154.94" y1="139.7" x2="152.4" y2="139.7" width="0.1524" layer="91"/>
+<label x="152.4" y="139.7" size="1.27" layer="95" rot="R180" xref="yes"/>
+</segment>
+<segment>
+<pinref part="R1" gate="G$1" pin="1"/>
+<wire x1="38.1" y1="152.4" x2="53.34" y2="152.4" width="0.1524" layer="91"/>
+<label x="53.34" y="152.4" size="1.27" layer="95" xref="yes"/>
+</segment>
+</net>
+<net name="PB2" class="0">
+<segment>
+<pinref part="U$2" gate="G$1" pin="LP_GPIO_15"/>
+<wire x1="154.94" y1="137.16" x2="152.4" y2="137.16" width="0.1524" layer="91"/>
+<label x="152.4" y="137.16" size="1.27" layer="95" rot="R180" xref="yes"/>
+</segment>
+<segment>
+<pinref part="R4" gate="G$1" pin="1"/>
+<wire x1="50.8" y1="149.86" x2="53.34" y2="149.86" width="0.1524" layer="91"/>
+<label x="53.34" y="149.86" size="1.27" layer="95" xref="yes"/>
+</segment>
+</net>
+<net name="I2C0_SCL" class="0">
+<segment>
+<pinref part="U$1" gate="G$1" pin="SWDIOALT"/>
+<wire x1="50.8" y1="53.34" x2="48.26" y2="53.34" width="0.1524" layer="91"/>
+<label x="48.26" y="53.34" size="1.27" layer="95" rot="R180" xref="yes"/>
+</segment>
+<segment>
+<wire x1="210.82" y1="60.96" x2="208.28" y2="60.96" width="0.1524" layer="91"/>
+<label x="210.82" y="60.96" size="1.27" layer="95" xref="yes"/>
+</segment>
+</net>
+<net name="I2C0_SDA" class="0">
+<segment>
+<pinref part="U$1" gate="G$1" pin="SWDCLKALT"/>
+<wire x1="50.8" y1="55.88" x2="48.26" y2="55.88" width="0.1524" layer="91"/>
+<label x="48.26" y="55.88" size="1.27" layer="95" rot="R180" xref="yes"/>
+</segment>
+<segment>
+<wire x1="210.82" y1="63.5" x2="208.28" y2="63.5" width="0.1524" layer="91"/>
+<label x="210.82" y="63.5" size="1.27" layer="95" xref="yes"/>
+</segment>
+</net>
+<net name="SWDCLK" class="0">
+<segment>
+<pinref part="U$1" gate="G$1" pin="SWDCLK"/>
+<wire x1="50.8" y1="60.96" x2="48.26" y2="60.96" width="0.1524" layer="91"/>
+<label x="48.26" y="60.96" size="1.27" layer="95" rot="R180" xref="yes"/>
+</segment>
+</net>
+<net name="SWDIO" class="0">
+<segment>
+<pinref part="U$1" gate="G$1" pin="SWDIO"/>
+<wire x1="50.8" y1="58.42" x2="48.26" y2="58.42" width="0.1524" layer="91"/>
+<label x="48.26" y="58.42" size="1.27" layer="95" rot="R180" xref="yes"/>
+</segment>
+</net>
+<net name="PB3" class="0">
+<segment>
+<pinref part="R5" gate="G$1" pin="1"/>
+<wire x1="38.1" y1="129.54" x2="53.34" y2="129.54" width="0.1524" layer="91"/>
+<label x="53.34" y="129.54" size="1.27" layer="95" xref="yes"/>
+</segment>
+<segment>
+<pinref part="U$1" gate="G$1" pin="P0.3"/>
+<wire x1="50.8" y1="38.1" x2="48.26" y2="38.1" width="0.1524" layer="91"/>
+<label x="48.26" y="38.1" size="1.27" layer="95" rot="R180" xref="yes"/>
+</segment>
+</net>
+<net name="PB4" class="0">
+<segment>
+<pinref part="R6" gate="G$1" pin="1"/>
+<wire x1="50.8" y1="127" x2="53.34" y2="127" width="0.1524" layer="91"/>
+<label x="53.34" y="127" size="1.27" layer="95" xref="yes"/>
+</segment>
+<segment>
+<pinref part="U$1" gate="G$1" pin="P0.2"/>
+<wire x1="50.8" y1="35.56" x2="48.26" y2="35.56" width="0.1524" layer="91"/>
+<label x="48.26" y="35.56" size="1.27" layer="95" rot="R180" xref="yes"/>
+</segment>
+</net>

Commit message: think I moved the pb's back to MAX32660 (using the i2c lines because they're not needed)
Connections:
- removed net I2C0_SCL: U$1.SWDIOALT
- removed net I2C0_SDA: U$1.SWDCLKALT
- net PB1: now also U$1.SWDCLKALT; no longer U$2.LP_GPIO_14
- net PB2: now also U$1.SWDIOALT; no longer U$2.LP_GPIO_15
Other:
- note added: "I will replace microusb w/ a tiny ckt (board2board?) will need to interface with debugger that has an actual microusb on it"
Changed lines of the file:
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@@
 <net name="PB1" class="0">
-<segment>
-<pinref part="U$2" gate="G$1" pin="LP_GPIO_14"/>
-<wire x1="154.94" y1="139.7" x2="152.4" y2="139.7" width="0.1524" layer="91"/>
-<label x="152.4" y="139.7" size="1.27" layer="95" rot="R180" xref="yes"/>
-</segment>
 <segment>
 <pinref part="R1" gate="G$1" pin="1"/>
@@
 <label x="53.34" y="152.4" size="1.27" layer="95" xref="yes"/>
 </segment>
+<segment>
+<pinref part="U$1" gate="G$1" pin="SWDCLKALT"/>
+<wire x1="50.8" y1="55.88" x2="48.26" y2="55.88" width="0.1524" layer="91"/>
+<label x="48.26" y="55.88" size="1.27" layer="95" rot="R180" xref="yes"/>
+</segment>
 </net>
 <net name="PB2" class="0">
-<segment>
-<pinref part="U$2" gate="G$1" pin="LP_GPIO_15"/>
-<wire x1="154.94" y1="137.16" x2="152.4" y2="137.16" width="0.1524" layer="91"/>
-<label x="152.4" y="137.16" size="1.27" layer="95" rot="R180" xref="yes"/>
-</segment>
 <segment>
 <pinref part="R4" gate="G$1" pin="1"/>
@@
 <label x="53.34" y="149.86" size="1.27" layer="95" xref="yes"/>
 </segment>
-</net>
-<net name="I2C0_SCL" class="0">
 <segment>
 <pinref part="U$1" gate="G$1" pin="SWDIOALT"/>
 <wire x1="50.8" y1="53.34" x2="48.26" y2="53.34" width="0.1524" layer="91"/>
 <label x="48.26" y="53.34" size="1.27" layer="95" rot="R180" xref="yes"/>
-</segment>
-<segment>
-<wire x1="210.82" y1="60.96" x2="208.28" y2="60.96" width="0.1524" layer="91"/>
-<label x="210.82" y="60.96" size="1.27" layer="95" xref="yes"/>
-</segment>
-</net>
-<net name="I2C0_SDA" class="0">
-<segment>
-<pinref part="U$1" gate="G$1" pin="SWDCLKALT"/>
-<wire x1="50.8" y1="55.88" x2="48.26" y2="55.88" width="0.1524" layer="91"/>
-<label x="48.26" y="55.88" size="1.27" layer="95" rot="R180" xref="yes"/>
-</segment>
-<segment>
-<wire x1="210.82" y1="63.5" x2="208.28" y2="63.5" width="0.1524" layer="91"/>
-<label x="210.82" y="63.5" size="1.27" layer="95" xref="yes"/>
 </segment>
 </net>
@@
 <sheet>
 <plain>
+<text x="185.42" y="104.14" size="1.27" layer="97">I will replace microusb w/
+a tiny ckt (board2board?)
+will need to interface with
+debugger that has an actual
+microusb on it</text>
 </plain>
 <instances>

Commit message: pretty much finished the board; swapped diode out for a smaller package
Parts:
- removed D2: PANASONIC_DB2J31400LPANASONIC_DB2J31400L_0_0, ringRemote:PANASONIC_DB2J31400LPANASONIC_DB2J31400L_0_0
- removed J1: AMPHENOL_10118192-0001LFAMPHENOL_10118192-0001LF_0_0, ringRemote:AMPHENOL_10118192-0001LFAMPHENOL_10118192-0001LF_0_0
- added U$6: 1X5_1.27MM, ringRemote:1X5_1.27MM
- added U$7: DB2731400L, ringRemote:DB2731400L
- D1: value RED -> ORANGE; device ringRemote:LED0603 -> ringRemote:LED0201
Connections:
- removed net D+: J1.3
- removed net D-: J1.2
- removed net VUSB: C7.1, J1.1, U$4.EN, U$4.IN
- new net VEXT: C7.1, U$4.EN, U$4.IN, U$6.2
- net GND: now also U$6.1; no longer J1.5, J1.MNT_1, J1.MNT_2, J1.MNT_3, J1.MNT_4, J1.MNT_5, J1.MNT_6
- net MAXRST: now also U$6.3
- net N$10: now also U$7.ANODE; no longer D2.ANODE
- net SWDCLK: now also U$6.5
- net SWDIO: now also U$6.4
- net VCC: now also U$7.CATHODE; no longer D2.CATHODE
Other:
- note removed: "I will replace microusb w/ a tiny ckt (board2board?) will need to interface with debugger that has an actual microusb on it"
Changed lines of the file:
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@@
 <layer number="59" name="tCarbon" color="7" fill="1" visible="no" active="no"/>
 <layer number="60" name="bCarbon" color="7" fill="1" visible="no" active="no"/>
-<layer number="88" name="SimResults" color="9" fill="1" visible="yes" active="yes"/>
+<layer number="88" name="SimResults" color="9" fill="1" visible="no" active="yes"/>
 <layer number="89" name="SimProbes" color="9" fill="1" visible="yes" active="yes"/>
 <layer number="90" name="Modules" color="5" fill="1" visible="yes" active="yes"/>
@@
 </classes>
 <parts>
-<part name="D1" library="ringRemote" deviceset="LED" device="0603" value="RED"/>
 <part name="Y1" library="ringRemote" deviceset="CRYSTAL-32.768KHZ" device="SMD-3.2X1.5" value="32.768kHz"/>
 <part name="C1" library="ringRemote" deviceset="CAPACITOR" device="" value="10uF"/>
@@
 <part name="U$4" library="ringRemote" deviceset="TLV700" device=""/>
 <part name="R7" library="ringRemote" deviceset="RESISTOR" device="0805" value="1.8k"/>
-<part name="D2" library="ringRemote" deviceset="PANASONIC_DB2J31400L" device="PANASONIC_DB2J31400L_0_0"/>
 <part name="U$5" library="ringRemote" deviceset="ML621S" device=""/>
 <part name="C7" library="ringRemote" deviceset="CAPACITOR" device="" value="1uF"/>
@@
 <part name="SUPPLY9" library="SparkFun-PowerSymbols" deviceset="VCC" device="" value="VCC"/>
 <part name="FRAME2" library="SparkFun-Aesthetics" deviceset="FRAME-LETTER" device="NO_PACKAGE"/>
-<part name="J1" library="ringRemote" deviceset="AMPHENOL_10118192-0001LF" device="AMPHENOL_10118192-0001LF_0_0"/>
-<part name="GND17" library="SparkFun-PowerSymbols" deviceset="GND2" device=""/>
-<part name="SUPPLY10" library="SparkFun-PowerSymbols" deviceset="VCC" device="" value="VUSB"/>
-<part name="SUPPLY11" library="SparkFun-PowerSymbols" deviceset="VCC" device="" value="VUSB"/>
+<part name="SUPPLY11" library="SparkFun-PowerSymbols" deviceset="VCC" device="" value="VEXT"/>
+<part name="U$6" library="ringRemote" deviceset="1X5_1.27MM" device=""/>
+<part name="D1" library="ringRemote" deviceset="LED" device="0201" value="ORANGE"/>
+<part name="U$7" library="ringRemote" deviceset="DB2731400L" device=""/>
 </parts>
 <sheets>
@@
 </plain>
 <instances>
-<instance part="D1" gate="G$1" x="99.06" y="22.86"/>
 <instance part="Y1" gate="G$1" x="142.24" y="114.3" smashed="yes" rot="R270">
 <attribute name="NAME" x="142.24" y="108.712" size="1.778" layer="95" font="vector" align="bottom-center"/>
@@
 <instance part="FRAME1" gate="G$1" x="0" y="0"/>
 <instance part="FRAME1" gate="V" x="147.32" y="0"/>
+<instance part="D1" gate="G$1" x="99.06" y="22.86"/>
 </instances>
 <busses>
@@
 </segment>
 <segment>
-<pinref part="D1" gate="G$1" pin="C"/>
 <pinref part="GND9" gate="G$1" pin="3.3V"/>
 <wire x1="99.06" y1="15.24" x2="99.06" y2="17.78" width="0.1524" layer="91"/>
+<pinref part="D1" gate="G$1" pin="C"/>
 </segment>
 <segment>
@@
 </segment>
 </net>
-<net name="N$5" class="0">
-<segment>
-<pinref part="R3" gate="G$1" pin="2"/>
-<pinref part="D1" gate="G$1" pin="A"/>
-</segment>
-</net>
 <net name="BT_RTS" class="0">
 <segment>
@@
 </segment>
 </net>
+<net name="N$5" class="0">
+<segment>
+<pinref part="R3" gate="G$1" pin="2"/>
+<pinref part="D1" gate="G$1" pin="A"/>
+</segment>
+</net>
 </nets>
 </sheet>
 <sheet>
 <plain>
-<text x="185.42" y="104.14" size="1.27" layer="97">I will replace microusb w/
-a tiny ckt (board2board?)
-will need to interface with
-debugger that has an actual
-microusb on it</text>
 </plain>
 <instances>
@@
 <instance part="U$4" gate="G$1" x="40.64" y="139.7"/>
 <instance part="R7" gate="G$1" x="78.74" y="134.62" rot="R90"/>
-<instance part="D2" gate="G$0" x="60.96" y="149.86"/>
 <instance part="U$5" gate="G$1" x="78.74" y="121.92" rot="R270"/>
 <instance part="C7" gate="G$1" x="15.24" y="139.7"/>
@@
 <instance part="FRAME2" gate="G$1" x="0" y="0"/>
 <instance part="FRAME2" gate="V" x="147.32" y="0"/>
-<instance part="J1" gate="G$0" x="144.78" y="134.62"/>
-<instance part="GND17" gate="G$1" x="170.18" y="101.6"/>
-<instance part="SUPPLY10" gate="G$1" x="170.18" y="124.46"/>
 <instance part="SUPPLY11" gate="G$1" x="15.24" y="149.86"/>
+<instance part="U$6" gate="G$1" x="187.96" y="91.44"/>
+<instance part="U$7" gate="G$1" x="60.96" y="149.86"/>
 </instances>
 <busses>
@@
 </segment>
 <segment>
-<pinref part="J1" gate="G$0" pin="5"/>
-<wire x1="162.56" y1="104.14" x2="165.1" y2="104.14" width="0.1524" layer="91"/>
-<pinref part="GND17" gate="G$1" pin="3.3V"/>
-<pinref part="J1" gate="G$0" pin="MNT_1"/>
-<wire x1="165.1" y1="104.14" x2="170.18" y2="104.14" width="0.1524" layer="91"/>
-<wire x1="162.56" y1="99.06" x2="165.1" y2="99.06" width="0.1524" layer="91"/>
-<wire x1="165.1" y1="99.06" x2="165.1" y2="93.98" width="0.1524" layer="91"/>
-<pinref part="J1" gate="G$0" pin="MNT_6"/>
-<wire x1="165.1" y1="93.98" x2="165.1" y2="88.9" width="0.1524" layer="91"/>
-<wire x1="165.1" y1="88.9" x2="165.1" y2="83.82" width="0.1524" layer="91"/>
-<wire x1="165.1" y1="83.82" x2="165.1" y2="78.74" width="0.1524" layer="91"/>
-<wire x1="165.1" y1="78.74" x2="165.1" y2="73.66" width="0.1524" layer="91"/>
-<wire x1="165.1" y1="73.66" x2="162.56" y2="73.66" width="0.1524" layer="91"/>
-<pinref part="J1" gate="G$0" pin="MNT_5"/>
-<wire x1="162.56" y1="78.74" x2="165.1" y2="78.74" width="0.1524" layer="91"/>
-<junction x="165.1" y="78.74"/>
-<pinref part="J1" gate="G$0" pin="MNT_4"/>
-<wire x1="162.56" y1="83.82" x2="165.1" y2="83.82" width="0.1524" layer="91"/>
-<junction x="165.1" y="83.82"/>
-<pinref part="J1" gate="G$0" pin="MNT_3"/>
-<wire x1="162.56" y1="88.9" x2="165.1" y2="88.9" width="0.1524" layer="91"/>
-<junction x="165.1" y="88.9"/>
-<pinref part="J1" gate="G$0" pin="MNT_2"/>
-<wire x1="162.56" y1="93.98" x2="165.1" y2="93.98" width="0.1524" layer="91"/>
-<junction x="165.1" y="93.98"/>
-<junction x="165.1" y="99.06"/>
-<wire x1="165.1" y1="99.06" x2="165.1" y2="104.14" width="0.1524" layer="91"/>
-<junction x="165.1" y="104.14"/>
-<label x="165.1" y="104.14" size="1.27" layer="95"/>
+<pinref part="U$6" gate="G$1" pin="1"/>
+<wire x1="195.58" y1="86.36" x2="198.12" y2="86.36" width="0.1524" layer="91"/>
+<label x="198.12" y="86.36" size="1.27" layer="95" xref="yes"/>
 </segment>
 </net>
@@
 <label x="38.1" y="101.6" size="1.27" layer="95" xref="yes"/>
 </segment>
+<segment>
+<pinref part="U$6" gate="G$1" pin="3"/>
+<wire x1="195.58" y1="91.44" x2="198.12" y2="91.44" width="0.1524" layer="91"/>
+<label x="198.12" y="91.44" size="1.27" layer="95" xref="yes"/>
+</segment>
 </net>
 <net name="N$10" class="0">
 <segment>
 <pinref part="U$4" gate="G$1" pin="OUT"/>
-<pinref part="D2" gate="G$0" pin="ANODE"/>
 <wire x1="53.34" y1="144.78" x2="58.42" y2="144.78" width="0.1524" layer="91"/>
+<pinref part="U$7" gate="G$1" pin="ANODE"/>
 </segment>
 </net>
 <net name="VCC" class="0">
 <segment>
-<pinref part="D2" gate="G$0" pin="CATHODE"/>
 <pinref part="R7" gate="G$1" pin="2"/>
 <wire x1="73.66" y1="144.78" x2="78.74" y2="144.78" width="0.1524" layer="91"/>
@@
 <junction x="78.74" y="144.78"/>
 <label x="78.74" y="144.78" size="1.27" layer="95" rot="R90"/>
+<pinref part="U$7" gate="G$1" pin="CATHODE"/>
 </segment>
 <segment>
@@
 </segment>
 </net>
-<net name="VUSB" class="0">
+<net name="VEXT" class="0">
 <segment>
 <pinref part="U$4" gate="G$1" pin="EN"/>
@@
 </segment>
 <segment>
-<pinref part="J1" gate="G$0" pin="1"/>
-<wire x1="162.56" y1="124.46" x2="170.18" y2="124.46" width="0.1524" layer="91"/>
-<pinref part="SUPPLY10" gate="G$1" pin="VCC"/>
-<label x="162.56" y="124.46" size="1.27" layer="95"/>
+<pinref part="U$6" gate="G$1" pin="2"/>
+<wire x1="195.58" y1="88.9" x2="198.12" y2="88.9" width="0.1524" layer="91"/>
+<label x="198.12" y="88.9" size="1.27" layer="95" xref="yes"/>
 </segment>
 </net>
@@
 </segment>
 </net>
-<net name="D-" class="0">
-<segment>
-<pinref part="J1" gate="G$0" pin="2"/>
-<wire x1="162.56" y1="119.38" x2="165.1" y2="119.38" width="0.1524" layer="91"/>
-<label x="165.1" y="119.38" size="1.27" layer="95" xref="yes"/>
-</segment>
-</net>
-<net name="D+" class="0">
-<segment>
-<pinref part="J1" gate="G$0" pin="3"/>
-<wire x1="162.56" y1="114.3" x2="165.1" y2="114.3" width="0.1524" layer="91"/>
-<label x="165.1" y="114.3" size="1.27" layer="95" xref="yes"/>
-</segment>
-</net>
+<net name="SWDCLK" class="0">
+<segment>
+<pinref part="U$6" gate="G$1" pin="5"/>
+<wire x1="195.58" y1="96.52" x2="198.12" y2="96.52" width="0.1524" layer="91"/>
+<label x="198.12" y="96.52" size="1.27" layer="95" xref="yes"/>
+</segment>
+</net>
+<net name="SWDIO" class="0">
+<segment>
+<pinref part="U$6" gate="G$1" pin="4"/>
+<wire x1="195.58" y1="93.98" x2="198.12" y2="93.98" width="0.1524" layer="91"/>
+<label x="198.12" y="93.98" size="1.27" layer="95" xref="yes"/>
+</segment>
+</net>

Commit message: tried to create some vias for the pushbuttons, these need to be routed offboard (past castellated edge near antenna section); created rev1 of mech model (this needs to be bigger and smoother, hurts my finger to wear right now)
Parts:
- removed C1: 10uF, ringRemote:CAPACITOR
- removed FRAME2: FRAME-LETTERNO_PACKAGE, SparkFun-Aesthetics:FRAME-LETTERNO_PACKAGE
- added C10, C9: 10uF, ringRemote:CAPACITOR-0402-16V-10%
- C5, C6: value 1uF -> 4pF
Connections:
- removed net VDDIO: C4.1, U$2.VDDIO
- net GND: now also C10.2, C9.2; no longer C1.2
- net VCC: now also C10.1, C4.1, C9.1, U$2.VDDIO; no longer C1.1
Other:
- note added: "so apparently the battery I chose can't supply enough current... so here's an extra cap?"
- note added: "use internal caps for tuning c5 and c6"
- note removed: "need to calculate c5 and c6 to match capacitance"
- note removed: "so apparently there are internal caps for tuning the crystal osc, so... can I be lazy and not include c5 and c6?"
